File: sata-backplane.kicad_sch (KiCad schematic)
At the start: 5 parts, among them J1 SATA_POWER_15, J10 SATA_1, J11 SATA_COMBINED_1, J20 SATA_2, J21 SATA_COMBINED_2

Commit message: Done, New parts & spacing
Parts:
- removed J1: SATA_POWER_15, sata:SATA_Power, symbol SATA:SATA_POWER_15
- removed J10: SATA_1, sata:SATA_Data, symbol SATA:SATA_DATA_7
- removed J11: SATA_COMBINED_1, sata:SATA_Combined, symbol SATA:SATA_COMBINED_22
- removed J20: SATA_2, sata:SATA_Data, symbol SATA:SATA_DATA_7
- removed J21: SATA_COMBINED_2, sata:SATA_Combined, symbol SATA:SATA_COMBINED_22
- added H1, H2, H3, H4: MountingHole_Pad, MountingHole:MountingHole_3.2mm_M3_Pad_TopBottom, symbol Mechanical:MountingHole_Pad
- added J1, J3: 470804001, CONN_47080-4001_MOL:CONN_47080-4001_MOL, symbol CONN_47080-4001_MOL:470804001
- added J2, J4: 877791001, CONN_877791001_MOL:CONN_877791001_MOL, symbol CONN_877791001_MOL:877791001
- added J5: SATA_POWER_15, sata:SATA_Power, symbol SATA:SATA_POWER_15
Connections:
- net GND: now also H1.1, H2.1, H3.1, H4.1, J1.1, J1.4, J1.7, J2.P10, J2.P12, J2.P4, J2.P5, J2.P6, J2.S1, J2.S4, J2.S7, J3.1, J3.4, J3.7, J4.P10, J4.P12, J4.P4, J4.P5, J4.P6, J4.S1, J4.S4, J4.S7, J5.10 (GND), J5.12 (GND), J5.4 (GND), J5.5 (GND), J5.6 (GND)
- net SATA1_A+: now also J1.2, J2.S2
- net SATA1_A-: now also J1.3, J2.S3
- net SATA1_B+: now also J1.5, J2.S5
- net SATA1_B-: now also J1.6, J2.S6
- net SATA2_A+: now also J3.2, J4.S2
- net SATA2_A-: now also J3.3, J4.S3
- net SATA2_B+: now also J3.5, J4.S5
- net SATA2_B-: now also J3.6, J4.S6
- new net 12V_A: J2.P14, J4.P14, J5.14 (V12)
- new net 12V_B: J2.P15, J4.P15, J5.15 (V12)
- new net 12V_PRE: J2.P13, J4.P13, J5.13 (V12)
- new net 3V3_A: J2.P1, J4.P1, J5.1 (V3.3)
- new net 3V3_B: J2.P2, J4.P2, J5.2 (V3.3)
- new net 5V_A: J2.P8, J4.P8, J5.8 (V5.0)
- new net 5V_B: J2.P9, J4.P9, J5.9 (V5.0)
- new net 5V_PRE: J2.P7, J4.P7, J5.7 (V5.0)
- new net PW_DIS: J2.P3, J4.P3, J5.3 (PWDIS)
- new net SS/ACT: J2.P11, J4.P11, J5.11 (ACT)
